File: hw/rev-b/cpu.kicad_sch (KiCad schematic)
At the start: 61 parts, among them J1 USB_C_Receptacle_USB2.0, J2 Micro_SD_Card_Det2, J3 DBG_UART, J4 Conn_01x06, SW1 SW_Push, SW2 SW_Push, U1 USBLC6-2P6, U2 W25Q16JVSSIQ, U3 RP2350_80QFN, U4 W956A8MBYA5I, U5 MCP79510, Y1 12MHz, Y2 32.768kHz

Commit message: schematic: radio sheet in the KiCad project (symbol lib generator, Croco edits applied + verified, PWR_FLAG, layout), KiCad lib env + re-recorded baseline, checker fixes (length-normalised fingerprints, accepted list, Radio sheet excluded from Croco netlist); logbook
Connections:
- net USB_D_prot+: no longer R9.2
- net USB_D_prot-: no longer R10.2
- new net USB_RP_D+: R9.2
- new net USB_RP_D-: R10.2
Changed lines of the file:
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@@
 		)
 	)
-	(global_label "USB_D_prot-"
+	(global_label "USB_RP_D-"
 		(shape input)
 		(at 254 77.47 0)
@@
 		)
 	)
-	(global_label "USB_D_prot+"
+	(global_label "USB_RP_D+"
 		(shape input)
 		(at 254 68.58 0)

Commit message: coin cell removed (DNP), RTC VBAT to GND per datasheet, power-symbol + dnp support in croco edit tool, board updated (BT1 off, +BATT ripped); logbook with save/RTC findings + correction
Parts:
- BT1: now not fitted; now left out of the parts list
Connections:
- net +BATT: no longer U5.3 (VBAT)
- net GND: now also U5.3 (VBAT)
Changed lines of the file:
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@@
 		(unit 1)
 		(exclude_from_sim no)
-		(in_bom yes)
-		(on_board yes)
-		(dnp no)
+		(in_bom no)
+		(on_board no)
+		(dnp yes)
 		(fields_autoplaced yes)
 		(property "Reference" "BT1"
@@
 	)
 	(symbol
-		(lib_id "power:+BATT")
+		(lib_id "power:GND")
 		(at 326.39 177.8 0)
 		(unit 1)
@@
 			)
 		)
-		(property "Value" "+BATT"
+		(property "Value" "GND"
 			(at 326.39 172.72 0)
 			(effects
@@
 			)
 		)
-		(property "Description" "Power symbol creates a global label with name \"+BATT\""
+		(property "Description" "Power symbol creates a global label with name \"GND\""
 			(at 326.39 177.8 0)
 			(effects

Commit message: J3/R11 debug UART header DNP + off board (ESP CS stub), free-space map counts placed new parts, sim: firmware-configured vs actual reservoir C, T520B reservoir runs
Parts:
- R11: now not fitted; now left out of the parts list
Changed lines of the file:
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@@
 		(exclude_from_sim no)
 		(in_bom no)
-		(on_board yes)
+		(on_board no)
 		(dnp yes)
 		(property "Reference" "J3"
@@
 		(unit 1)
 		(exclude_from_sim no)
-		(in_bom yes)
-		(on_board yes)
-		(dnp no)
+		(in_bom no)
+		(on_board no)
+		(dnp yes)
 		(property "Reference" "R11"
 			(at 363.22 114.1222 90)

Commit message: JLC order files: BOM (live-checked, 3 out-of-stock Croco chips replaced, C27/C28 value fix), CPL with pad-matched rotations/offsets, Gerbers+drill, ORDER.md; gate PASS
Parts:
- C27: value 4.3.pF -> 4.3pF; LCSC C1644 -> C59526
- C28: LCSC C1644 -> C59526
- U1: LCSC C15999 -> C2827693
- U2: value W25Q16JVSSIQ -> W25Q128JVSIQ; LCSC C82317 -> C97521
- U4: value W956A8MBYA5I -> IS66WVH8M8BLL-100B1LI; LCSC C5375118 -> C1349096
Changed lines of the file:
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@@
 			)
 		)
-		(property "LCSC" "C15999"
+		(property "LCSC" "C2827693"
 			(at 35.56 102.87 90)
 			(effects
@@
 			)
 		)
-		(property "Value" "4.3.pF"
+		(property "Value" "4.3pF"
 			(at 347.853 186.309 0)
 			(effects
@@
 			)
 		)
-		(property "LCSC" "C1644"
+		(property "LCSC" "C59526"
 			(at 346.71 189.23 0)
 			(effects
@@
 			)
 		)
-		(property "Value" "W956A8MBYA5I"
+		(property "Value" "IS66WVH8M8BLL-100B1LI"
 			(at 205.2194 240.1371 0)
 			(effects
@@
 			)
 		)
-		(property "Datasheet" "https://www.winbond.com/resource-files/W958D8NBYA%20256Mb%20HyperRAM%20TFBGA24%20SDP%2085C%20datasheet_A01-002_20211020.pdf"
+		(property "Datasheet" "https://www.issi.com/WW/pdf/66-67WVH8M8ALL-BLL.pdf"
 			(at 191.77 237.49 0)
 			(effects
@@
 			)
 		)
-		(property "LCSC" "C5375118"
+		(property "LCSC" "C1349096"
 			(at 200.66 256.54 0)
 			(effects
@@
 			)
 		)
-		(property "LCSC" "C1644"
+		(property "LCSC" "C59526"
 			(at 346.71 198.12 0)
 			(effects
@@
 			)
 		)
-		(property "Value" "W25Q16JVSSIQ"
+		(property "Value" "W25Q128JVSIQ"
 			(at 71.8694 161.3971 0)
 			(effects
@@
 			)
 		)
-		(property "LCSC" "C82317"
+		(property "LCSC" "C97521"
 			(at 69.85 170.18 0)
 			(effects
