File: hw/rev-b/cpu.kicad_sch (KiCad schematic)
At the start: 61 parts, among them J1 USB_C_Receptacle_USB2.0, J2 Micro_SD_Card_Det2, J3 DBG_UART, J4 Conn_01x06, SW1 SW_Push, SW2 SW_Push, U1 USBLC6-2P6, U2 W25Q128JVSIQ, U3 RP2350_80QFN, U4 IS66WVH8M8BLL-100B1LI, U5 MCP79510, Y1 12MHz, Y2 32.768kHz

Commit message: Rev B: fixes from the wallet cart's JLC check and datasheet review
- JLC gate (verify/jlc_check.py): top-edge GND vias 0.06 mm inward, copper-to-edge
  rule 0.2 mm with a J5 exemption (.kicad_dru), back URL/credit text 1.0 mm. PASS.
- Radio-area ground: F.Cu GND pour, 56 stitching vias, one via per U104 centre
  sub-pad, vias at U103 GND pins, C106, U106.4. GND vias 214 -> 285.
- RP2350 VREG_LX keepout on In1-In4; DEBUG_UART_TX and LED_DIN rerouted around it.
- R110 -> C453777 (C4147 below JLC's minimum buy); make_bom now checks minimum buy.
- R133 4.7k GBBUS_EN pull-down (TXB0108 OE).
- Y1 -> ABM8-272-T3 C20625731.
- USB upstream D+ moved onto In2 with D-: 2 vias each, 12.42 / 11.84 mm.
- All gates re-run; BOM/CPL/Gerbers/zip/renders regenerated. LOGBOOK 2026-10-16 12:15.

Co-Authored-By: Claude Opus 5.5 (1M context) <noreply@anthropic.com>
Claude-Session: https://claude.ai/code/session_01F5zMMQgMFiMCad54U85DYT
Parts:
- Y1: LCSC C668845 -> C20625731
Changed lines of the file:
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@@
 			)
 		)
-		(property "LCSC" "C668845"
+		(property "LCSC" "C20625731"
 			(at 148.59 125.73 90)
 			(effects
